File: kicad/serge-gain-cell.kicad_sch (KiCad schematic)
At the start: 21 parts, among them J2 Conn_01x04_Pin, J3 Conn_01x04_Pin, Q1 2N3904, Q2 2N3906, Q3 2N3904, Q4 2N3906, U1 LF353

Commit message: Updating to newer kicad version
Parts:
- C3, C4: Spec ceramic C0G -> ceramic X7R
